File: fm_vevo.kicad_pcb (KiCad board)
At the start: 2 copper layers, 87.5 x 47.5 mm, 89 parts, among them J1 RedPitaya_kimenete, J2 bemenet2, J3 Bemenet, J4 RedPitaya_+-10V, J5 12VDC, J6 RedPitaya_+-1V, J7 AudioJack, Q1 mmbfj310, Q2 MMBT3904, U1 LM358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

Commit message: Silkscreen
Parts:
- J1: value RedPitaya_kimenete -> Hang. fesz.
- J4: value RedPitaya_+-10V -> HO/1024
- moved H1 0.62 mm to (24.9, 50.0)
Other:
- board text added: "FM vevő"

Commit message: Silk
Other:
- board text added: "2020 tavasz"
- board text added: "A koronavírus járvány alatt tartott távfoglalkozások eredménye"

Commit message: Silk
Parts:
- J1: value Hang. fesz. -> Hangoló fesz.
Changed lines of the file:
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@@
     (35 F.Paste user hide)
     (36 B.SilkS user)
-    (37 F.SilkS user hide)
+    (37 F.SilkS user)
     (38 B.Mask user)
     (39 F.Mask user hide)
@@
       (effects (font (size 1 1) (thickness 0.15)))
     )
-    (fp_text value "Hang. fesz." (at 1.002 9.994 180) (layer F.SilkS)
-      (effects (font (size 1 1) (thickness 0.15)))
-    )
+    (fp_text value "Hangoló fesz." (at 1.002 11.244 180) (layer F.SilkS)
+      (effects (font (size 1 1) (thickness 0.15)))
+    )

Commit message: TBA120S demodulator added
Other:
- board text added: "JLCJLCJLCJLC"
